File: C64 1541-II ROM Adapter/C64 1541-II ROM Adapter.sch (KiCad schematic (older format))
At the start: 7 parts, among them J1 A14, J2 A15, J3 GND, U1 27C512

Commit message: Shorten ROM board a little bit
Parts:
- J1, J2, J3: footprint edge_connect:edge_pins_1x01 -> edge_connect:short_edge_pins_1x01
Changed lines of the file:
@@
 F 0 "J3" H 9147 3832 50  0000 R CNN
 F 1 "GND" H 9147 3923 50  0000 R CNN
-F 2 "edge_connect:edge_pins_1x01" H 9175 3900 50  0001 C CNN
+F 2 "edge_connect:short_edge_pins_1x01" H 9175 3900 50  0001 C CNN
 F 3 "~" H 9175 3900 50  0001 C CNN
 	1    9175 3900
@@
 F 0 "J1" H 9147 3432 50  0000 R CNN
 F 1 "A14" H 9147 3523 50  0000 R CNN
-F 2 "edge_connect:edge_pins_1x01" H 9175 3500 50  0001 C CNN
+F 2 "edge_connect:short_edge_pins_1x01" H 9175 3500 50  0001 C CNN
 F 3 "~" H 9175 3500 50  0001 C CNN
 	1    9175 3500
@@
 F 0 "J2" H 9147 3632 50  0000 R CNN
 F 1 "A15" H 9147 3723 50  0000 R CNN
-F 2 "edge_connect:edge_pins_1x01" H 9175 3700 50  0001 C CNN
+F 2 "edge_connect:short_edge_pins_1x01" H 9175 3700 50  0001 C CNN
 F 3 "~" H 9175 3700 50  0001 C CNN
 	1    9175 3700
