File: C64 XUM1541-II/C64 XUM1541-II.sch (KiCad schematic (older format))
At the start: 19 parts, among them J1 IEC, J2 PARALLEL, M1 Mounting, M2 Mounting, M3 Mounting, M4 Mounting, SW1 RESET, U1 7406

Commit message: Resistor note
Other:
- note added: "The resistor values here are\nmore of a suggestion, just\nto keep them from burning\nout.\n\nBright LEDs might not be\ncomfortable to look at with\nthis value, for those I'd\nconsider something up to 3k3.\nEither calculate from datasheet\nor test on a breadboard before\nsoldering."
Changed lines of the file:
@@
 	3725 6175 1575 6175
 Wire Notes Line
-	10200 1600 10200 2825
+	10975 1600 10975 2825
 Text Notes 8825 1575 0    60   ~ 0
 LED indicators (optional)
@@
 Wire Notes Line
 	8800 2825 8800 1600
-Wire Notes Line
-	8800 1600 10200 1600
-Wire Notes Line
-	8800 2825 10200 2825
 Text Notes 8825 3150 0    60   ~ 0
 Arduino reset (optional)
@@
 Wire Wire Line
 	5800 1650 5875 1650
+Text Notes 9975 2575 0    39   ~ 0
+The resistor values here are\nmore of a suggestion, just\nto keep them from burning\nout.\n\nBright LEDs might not be\ncomfortable to look at with\nthis value, for those I'd\nconsider something up to 3k3.\nEither calculate from datasheet\nor test on a breadboard before\nsoldering.
+Wire Notes Line
+	8800 2825 10975 2825
+Wire Notes Line
+	8800 1600 10975 1600
 Wire Bus Line
 	4750 1000 4750 2050
